File: filter01/filter01.kicad_pcb (KiCad board)
At the start: 2 copper layers, 10.8 x 12.7 mm, 10 parts, among them J1 Conn_01x01_Female, J2 Conn_01x01_Female, J3 Conn_01x01_Female, J4 Conn_01x01_Female, J5 Conn_01x01_Female, J6 Conn_01x01_Female

Commit message: Fixed issued
Parts:
- turned J1 to 180 degrees
Routing:
- net GND: vias 0 -> 9
- net (no net): vias 9 -> 0
Other:
- board size 10.8 x 12.7 mm -> 10.8 x 14 mm
Changed lines of the file:
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@@
     (user_trace_width 0.5)
     (trace_clearance 0.2)
-    (zone_clearance 0.15)
+    (zone_clearance 0.4)
     (zone_45_only no)
     (trace_min 0.2)
@@
   )
   (module Connector_Wire:SolderWirePad_1x01_SMD_1x2mm (layer B.Cu)
-    (at 195.58 72.39 270)
+    (at 195.58 72.39 180)
     (descr "Wire Pad, Square, SMD Pad,  5mm x 10mm,")
     (tags "MesurementPoint Square SMDPad 5mmx10mm ")
     (attr virtual)
-    (fp_text reference J1 (at 0 2.54 270) (layer B.SilkS)
-      (effects (font (size 1 1) (thickness 0.15)) (justify mirror))
-    )
-    (fp_text value Conn_01x01_Female (at 0 -2.54 270) (layer B.Fab)
+    (fp_text reference J1 (at 0 2.54 180) (layer B.SilkS)
+      (effects (font (size 1 1) (thickness 0.15)) (justify mirror))
+    )
+    (fp_text value Conn_01x01_Female (at 0 -2.54 180) (layer B.Fab)
       (effects (font (size 1 1) (thickness 0.15)) (justify mirror))
     )
@@
     (fp_line (start 0.63 -1.27) (end 0.63 1.27) (layer B.CrtYd) (width 0.05))
     (fp_line (start 0.63 1.27) (end -0.63 1.27) (layer B.CrtYd) (width 0.05))
-    (fp_text user %R (at 0 0 270) (layer B.Fab)
-      (effects (font (size 1 1) (thickness 0.15)) (justify mirror))
-    )
-    (pad 1 smd roundrect (at 0 0 270) (size 1 2) (layers B.Cu B.Paste B.Mask) (roundrect_rratio 0.25)
+    (fp_text user %R (at 0 0 180) (layer B.Fab)
+      (effects (font (size 1 1) (thickness 0.15)) (justify mirror))
+    )
+    (pad 1 smd roundrect (at 0 0 180) (size 1 2) (layers B.Cu B.Paste B.Mask) (roundrect_rratio 0.25)
       (net 4 GND))
   )
@@
     (arrow2b (pts (xy 210.82 59.69) (xy 211.406421 60.816504)))
   )
-  (gr_line (start 202.565 59.69) (end 202.565 72.39) (layer Edge.Cuts) (width 0.1))
+  (gr_line (start 202.565 59.69) (end 202.565 73.66) (layer Edge.Cuts) (width 0.1))
   (gr_line (start 191.77 59.69) (end 202.565 59.69) (layer Edge.Cuts) (width 0.1))
-  (gr_line (start 191.77 72.39) (end 191.77 59.69) (layer Edge.Cuts) (width 0.1))
-  (gr_line (start 202.565 72.39) (end 191.77 72.39) (layer Edge.Cuts) (width 0.1))
-  (via (at 201.93 60.325) (size 0.8) (drill 0.4) (layers F.Cu B.Cu) (net 0))
-  (via (at 192.405 60.325) (size 0.8) (drill 0.4) (layers F.Cu B.Cu) (net 0))
-  (via (at 192.405 62.23) (size 0.8) (drill 0.4) (layers F.Cu B.Cu) (net 0))
-  (via (at 192.405 64.135) (size 0.8) (drill 0.4) (layers F.Cu B.Cu) (net 0))
-  (via (at 192.405 66.675) (size 0.8) (drill 0.4) (layers F.Cu B.Cu) (net 0))
-  (via (at 201.93 62.865) (size 0.8) (drill 0.4) (layers F.Cu B.Cu) (net 0))
-  (via (at 201.93 65.405) (size 0.8) (drill 0.4) (layers F.Cu B.Cu) (net 0))
-  (via (at 199.39 60.325) (size 0.8) (drill 0.4) (layers F.Cu B.Cu) (net 0))
-  (via (at 201.93 69.85) (size 0.8) (drill 0.4) (layers F.Cu B.Cu) (net 0))
+  (gr_line (start 191.77 73.66) (end 191.77 59.69) (layer Edge.Cuts) (width 0.1))
+  (gr_line (start 202.565 73.66) (end 191.77 73.66) (layer Edge.Cuts) (width 0.1))
+  (via (at 201.93 60.325) (size 0.8) (drill 0.4) (layers F.Cu B.Cu) (net 4))
+  (via (at 192.405 60.325) (size 0.8) (drill 0.4) (layers F.Cu B.Cu) (net 4))
+  (via (at 192.405 62.23) (size 0.8) (drill 0.4) (layers F.Cu B.Cu) (net 4))
+  (via (at 192.405 64.135) (size 0.8) (drill 0.4) (layers F.Cu B.Cu) (net 4))
+  (via (at 192.405 66.675) (size 0.8) (drill 0.4) (layers F.Cu B.Cu) (net 4))
+  (via (at 201.93 62.865) (size 0.8) (drill 0.4) (layers F.Cu B.Cu) (net 4))
+  (via (at 201.93 65.405) (size 0.8) (drill 0.4) (layers F.Cu B.Cu) (net 4))
+  (via (at 199.39 60.325) (size 0.8) (drill 0.4) (layers F.Cu B.Cu) (net 4))
+  (via (at 201.93 69.85) (size 0.8) (drill 0.4) (layers F.Cu B.Cu) (net 4))
   (segment (start 199.87 69.85) (end 200.66 69.85) (width 0.5) (layer F.Cu) (net 1))
   (segment (start 200.66 67.515) (end 200.865 67.31) (width 0.5) (layer F.Cu) (net 1))
@@
   (segment (start 195.58 67.115) (end 197.72 67.115) (width 0.5) (layer F.Cu) (net 3))
   (segment (start 195.58 64.965) (end 195.58 60.96) (width 0.5) (layer F.Cu) (net 5))
-  (zone (net 4) (net_name GND) (layer F.Cu) (hatch edge 0.508)
-    (connect_pads (clearance 0.15))
-    (min_thickness 0.1)
-    (fill yes (arc_segments 32) (thermal_gap 0.15) (thermal_bridge_width 0.15))
+  (zone (net 4) (net_name GND) (layer B.Cu) (hatch edge 0.508)
+    (connect_pads (clearance 0.2))
+    (min_thickness 0.2)
+    (fill yes (arc_segments 32) (thermal_gap 0.508) (thermal_bridge_width 0.508))
     (polygon
       (pts
-        (xy 202.565 72.39) (xy 191.77 72.39) (xy 191.77 59.69) (xy 202.565 59.69)
+        (xy 203.2 73.66) (xy 191.77 73.66) (xy 191.77 59.69) (xy 203.2 59.69)
       )
     )
   )
-  (zone (net 4) (net_name GND) (layer B.Cu) (hatch edge 0.508)
-    (connect_pads (clearance 0.2))
+  (zone (net 4) (net_name GND) (layer F.Cu) (hatch edge 0.508)
+    (connect_pads (clearance 0.4))
     (min_thickness 0.1)
-    (fill yes (arc_segments 32) (thermal_gap 0.15) (thermal_bridge_width 0.15))
+    (fill yes (arc_segments 32) (thermal_gap 0.508) (thermal_bridge_width 0.508))
     (polygon
       (pts
-        (xy 202.565 72.39) (xy 191.77 72.39) (xy 191.77 59.69) (xy 202.565 59.69)
+        (xy 203.2 73.66) (xy 191.77 73.66) (xy 191.77 59.69) (xy 203.2 59.69)
       )
     )
